Commit message: fix material

File: ct_models/urdf/HyQ/links/leg.urdf.xacro (robot description, xacro)
@@ -105,5 +105,7 @@
 					<mesh filename="package://ct_models/urdf/HyQ/meshes/leg/lowerleg.dae" scale="1 1 1"/>
 				</geometry>
-				<material name="white"/>
+      <material name="White">
+        <color rgba="1.0 1.0 1.0 1.0"/>
+      </material>
 			</visual>
 			<collision>
